File: projects/HALLICRAFTERS S-38A/HALLICRAFTERS S-38A.kicad_sch (KiCad schematic)
At the start: 22 parts, among them P1 Conn_WallPlug, SW1 PART OF R7

Commit message: LOTS OF ADDS
Parts:
- added C1, C10, C2, C3, C4, C7, C8, C9: C_Variable, symbol Device:C_Variable
- added C11, C12, C13, C14, C15, C17, C5, C6: 0.25uf, symbol Device:C_Small
- added C16, C30: 0.02uf, symbol Device:C_Small
- added C18: .25uf, symbol Device:C_Small
- added C19: .02uf, symbol Device:C_Small
- added C20: 0.05uf, symbol Device:C_Small
- added C24A: 5000, symbol Device:C_Small
- added C24B, C24C: 220, symbol Device:C_Small
- added C24D: 2000, symbol Device:C_Small
- added C29A: 20uf, symbol Device:C_Small
- added C40: 0.01uf, symbol Device:C_Small
- added C41, C42: GIMMIK, symbol Device:C_Small
- added C7A, C7A1, C7B, C7B1: C_TRIMMER, symbol Vintage_Radio_Passives:C_TRIMMER
- added F1: Fuse, symbol Device:Fuse
- added L1, L2, L3, L4, L5, L6, L7: COIL, symbol Vintage_Radio_Transformers_Coils:COIL_5_TAP
- added L10, L11, L8, L9: COIL, symbol Vintage_Radio_Transformers_Coils:COIL_4_TAP
- added L12: COIL, symbol Vintage_Radio_Transformers_Coils:COIL_2_TAP
- added LM2: ~, symbol Vintage_Radio_Passives:LAMP
- added LS1: ~, symbol Vintage_Radio_Transformers_Coils:SPEAKER
- added P3: Conn_WallPlug_Earth, symbol Connector:Conn_WallPlug_Earth
- added R1, R2: 22K, symbol Device:R_US
- added R10: 10K, symbol Device:R_US
- added R11: 330, symbol Device:R_US
- added R12: 220K, symbol Device:R_US
- added R13, R20: 470K, symbol Device:R_US
- added R14: 150, symbol Device:R_US
- added R15: 15, symbol Device:R_US
- added R21: 22, symbol Device:R_US
- added R3, R9: 470, symbol Device:R_US
- added R4: 390, symbol Device:R_US
- added R5: 2.2M, symbol Device:R_US
- added R6: 47K, symbol Device:R_US
- added R7: 500K, symbol Device:R_Potentiometer_US
- added R8: 10M, symbol Device:R_US
- added S1: ON/OFF, symbol Switch:SW_SPST
- added S1A, S1D: SW_SPST, symbol Vintage_Radio_Passives:ROTARY_SW_1P4T
- added S1B, S1C: ~, symbol Vintage_Radio_Switches:ROTARY_SW_1P5T_X
- added S3, SW2: SW_SPDT, symbol Vintage_Radio_Switches:SW_SPDT
- added SW2: RCV/STBY, symbol Switch:SW_SPST
- added T4, T5: 455 kHz, symbol Vintage_Radio_Transformers_Coils:IF_XFMR
- added T6: OUTPUT, symbol Vintage_Radio_Transformers_Coils:OUTPUT TRANSFORMER
- added TS1: ANTENNA, symbol Connector:Screw_Terminal_01x03
- added TS2: PHONES, symbol Connector:Screw_Terminal_01x02
- added V10: 35Z5GT, Vintage_Radio_Vacuum_Tubes:Octal Socket - THT, symbol Vintage_Radio_Vacuum_Tubes:35Z5GT
- added V6, V7, V8, V9: ~, symbol Vintage_Radio_Vacuum_Tubes:HEATER
- SW1: value PART OF R7 -> ON/OFF
- V2: renamed from V3; value 12SG7 -> 12SK7
- renumbered V2 to V1, V4 to V3, V5 to V4
Connections:
- net GNDREF: now also C10.2, C11.2, C16.2, C17.2, C18.1, C19.2, C20.2, C24B.1, C24C.1, C29A.2, C30.2, C5.2, C6.2, C7.2, C7A.2, C7A1.2, C7B.2, C7B1.2, C8.2, C9.2, P3.2 (AC_N), R13.1, R14.1, R2.1, R20.1, R3.1, R7.1, R8.2, S1C.1 (A), S3.2 (B), SW2.1 (A), V6.8
- net at C29D.1, R16.2: now also C11.1, C17.1, L12.1, R12.1, T4.2, T5.2
- net at C29C.1, R16.1, R17.2: now also T6.2
- net GNDPWR renamed CASE
- net CASE: now also C18.2, P3.3 (EARTH)
- new net: C13.2, C7.1, L8.1
- new net: L8.2, S1D.1 (A)
- new net: L1.1, R10.2, S1A.1 (A)
- new net: L1.2, L2.2, L3.2, R10.1, TS1.2 (Pin_2)
- new net: F1.1, P3.1 (AC_P)
- new net: F1.2, S1.2 (B)
- new net: C14.1, C7A1.1, C7B1.1
- new net: C4.1, L7.1, S1B.1 (A)
- new net: C4.2, C6.1, L7.2, R3.2
- new net: C24D.1, R8.1
- new net: C24D.2, R7.2
- new net: C29A.1, R14.2
- new net: C24A.1, R13.2
- new net: C24A.2, C24B.2, R12.2
- new net: C12.2, C8.1, L9.1
- new net: L9.2, S1D.1 (A)
- new net: V7.8, V8.7
- new net: V8.8, V9.7
- new net: C12.1, S1C.1 (A)
- new net: L12.2, R21.1
- new net: C9.1, L10.1, S1C.1 (A)
- new net: C1.2, C16.1, C2.2, C3.2, L4.2, L5.2, L6.2, R5.2, R9.2, S1B.1 (A), T4.3
- new net: C7A.1, C7B.1, S1B.1 (A)
- new net: C2.1, L5.1, S1B.1 (A)
- new net: C1.1, L4.1, S1B.1 (A)
- new net: C3.1, L6.1, S1B.1 (A)
- new net: LM2.1, R11.2
- new net: C19.1, LM2.2, R11.1, S1.1 (A)
- new net: V6.7, V7.7
- new net: R9.1, S3.3 (C)
- new net: C10.1, L11.1, S1C.1 (A)
- new net: C15.2, R2.2
- new net: C13.1, S1C.1 (A)
- new net: C14.2, R1.1, S1C.1 (A)
- new net: C15.1, R1.2
- new net: L3.1, S1A.1 (A)
- new net: S1A.1 (A), TS1.3 (Pin_3)
- new net: L2.1, S1A.1 (A)
- new net: R15.1, SW2.1 (A), TS2.2 (Pin_2)
- new net: SW2.2 (B), T6.3
- new net: LS1.1, SW2.3 (C)
- new net: C41.1, T4.4
- new net: C5.1, TS1.1 (Pin_1)
- new net: C42.1, T5.1
- new net: C41.2, C42.2, S3.1 (A)
- new net: R15.2, T6.4, TS2.1 (Pin_1)
- new net: C40.1, R7.3
- new net: C40.2, R20.2, R5.1, R6.1
- new net: C24C.2, R6.2, T5.3
- new net: C20.1, R4.2
- new net: L11.2, S1D.1 (A)
- new net: C30.1, T6.1
- new net: LS1.2, T6.5
- new net: L10.2, S1D.1 (A)
- new net: R4.1, SW2.2 (B)
Other:
- note added: "10"
- note added: "11"
- note added: "12"
- note added: "13"
- note added: "14"
- note added: "15"
- note added: "16"
- note added: "18"
- note added: "19"
- note added: "2"
- note added: "20"
- note added: "21"
- note added: "22"
- note added: "23"
- note added: "24"
- note added: "25"
- note added: "26"
- note added: "27"
- note added: "3"
- note added: "4"
- note added: "5"
- note added: "6"
- note added: "7"
- note added: "8"
- note added: "9"
- note added: "A"
- note added: "A1"
- note added: "A2"
- note added: "AM"
- note added: "B"
- note added: "C"
- note added: "CW"
- note added: "D"
- note added: "F"
- note added: "G"
- note added: "M"
- note added: "N"
- note added: "O"
- note added: "P"
- note added: "Q"
- note added: "T1"
- moved on the sheet: C29B, C29C, C29D, C34, C36, C39, LM1, P1, R16, R17, R18, R19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

Commit message: MORE CHANGES
Parts:
- F1: value Fuse -> 1 AMP
- renumbered P3 to PL1
Connections:
- net at F1.2: now also S1.1 (A); no longer S1.2 (B)
- net at C19.1, LM2.2, R11.1: now also S1.2 (B); no longer S1.1 (A)
- net at S1D.1 (A): now also L10.2
Other:
- note added: "1. CHANGE TO 3 PIN AC PLUG 2. ADD FUSE 3. MOVE SWITCH TO LINE SIDE 4. PLUG GROUND TO CASE"
- note added: "SAFETY MODIFICATION FOR PROPER GROUNDING"
- moved on the sheet: C18, C19, F1, LM2, PL1, R11, S1, V10, V6, V7, V8, V9

Commit message: MULTIPLE VALUE CHANGES
Parts:
- removed C13: 0.25uf, symbol Device:C_Small
- removed C19: .02uf, symbol Device:C_Small
- removed LM2: ~, symbol Vintage_Radio_Passives:LAMP
- added C10: C_Variable, symbol Device:C_Variable
- C1: renamed from C5; value 0.25uf -> 0.01uf
- C11: renamed from C12; value 0.25uf -> 2200pf
- C24A: value 5000 -> 5000pf
- C24B, C24C: value 220 -> 220pf
- C24D: value 2000 -> 2000pf
- C34: value .02uf -> 0.02uf
- C36: value .25uf -> 0.25uf
- C36: renamed from C18; value .25uf -> 0.25uf
- C6: value 0.25uf -> 2200pf
- C8: renamed from C15; value 0.25uf -> 220pf
- C9: renamed from C14; value 0.25uf -> 3000pf
- R3: value 470 -> 470K
- R3: renamed from R1; value 22K -> 47
- renumbered C7 to C12, C8 to C13, C9 to C14, C10 to C15, C1 to C2, C2 to C3, C3 to C4, C4 to C5, C7A1 to C7C, C7B1 to C7D, P1 to PL1, SW1 to S1, SW2 to S4
Connections:
- net GNDREF: now also C41.2, C42.2, S1D.1 (A), S3.1 (A)
- net at C12.1, L8.1: now also C10.1
- new net: C10.2, S1C.1 (A)
Other:
- note added: "GANGED WITH C7A"
- note added: "GANGED WITH C7B"
- note added: "GANGED WITH C7C"
- note added: "GANGED WITH C7D"
- note added: "H"
- note added: "I"
- note added: "K"
- note added: "L"
- note added: "PHONES"
- note added: "S"
- note added: "SAFETY MODIFICATION"
- note added: "SPEAKER"
- note added: "T"
- note added: "T2"
- note added: "T3"
- note added: "U"
- note added: "V"
- note added: "W"
- note removed: "SAFETY MODIFICATION FOR PROPER GROUNDING"
- company: (none) -> K4TFJ Projects
- title: (none) -> Hallicrafters S-38A Schematic
- moved on the sheet: C1, C11, C12, C13, C14, C15, C16, C17, C2, C20, C24A, C24B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
